File: V2/electronics/main/main.kicad_sch (KiCad schematic)
At the start: 4 parts

Commit message: main sch layout 04 04 22
Parts:
- removed J?: USB_B_Micro, Connector_USB:USB_Micro-B_Molex-105017-0001, symbol Connector:USB_B_Micro
- removed SW?: PWR MFB, TL3365_button:TL3365_button, symbol Switch:SW_Push
- removed SW?: RESET, TL3365_button:TL3365_button, symbol Switch:SW_Push
- added C? (x3): 10µF, 0805-NO, symbol Adafruit Feather M0 Basic rev C-eagle-import:CAP_CERAMIC0805-NOOUTLINE
- added C?: 0.1uF, 0805_10MGAP, symbol Adafruit MPR121 Breakout-eagle-import:CAP_CERAMIC0805_10MGAP
- added C?: 10µF, _0805MP, symbol Adafruit VS1053 Headphone FeatherWing-eagle-import:CAP_CERAMIC_0805MP
- added C? (x2): 22pF, 0603-NO, symbol Adafruit VS1053 Headphone FeatherWing-eagle-import:CAP_CERAMIC0603_NO
- added C? (x2): 220uF, PANASONIC_C, symbol Adafruit VS1053 Headphone FeatherWing-eagle-import:CPOL-USC
- added C?: 0.1µF, 0603-NO, symbol Adafruit VS1053 Headphone FeatherWing-eagle-import:CAP_CERAMIC0603_NO
- added C?: 0.1uF, 0805-NO, symbol Adafruit MPR121 Breakout-eagle-import:CAP_CERAMIC0805-NOOUTLINE
- added C?: 10uF, 0805-NO, symbol Adafruit Feather M0 Basic rev C-eagle-import:CAP_CERAMIC0805-NOOUTLINE
- added C? (x2): 1µF, 0603-NO, symbol Adafruit VS1053 Headphone FeatherWing-eagle-import:CAP_CERAMIC0603_NO
- added C? (x2): 22pF, 0603-NO, symbol Adafruit Feather M0 Basic rev C-eagle-import:CAP_CERAMIC0603_NO
- added C? (x3): 1uF, 0603-NO, symbol Adafruit Feather M0 Basic rev C-eagle-import:CAP_CERAMIC0603_NO
- added C? (x2): 10nF, 0603-NO, symbol Adafruit VS1053 Headphone FeatherWing-eagle-import:CAP_CERAMIC0603_NO
- added C?: 10µF, 0805-NO, symbol Adafruit VS1053 Headphone FeatherWing-eagle-import:CAP_CERAMIC0805-NOOUTLINE
- added C?: 1uF, 0603-NO, symbol Adafruit VS1053 Headphone FeatherWing-eagle-import:CAP_CERAMIC0603_NO
- added CHG?: ORANGE, CHIPLED_0805_NOOUTLINE, symbol Adafruit Feather M0 Basic rev C-eagle-import:LED0805_NOOUTLINE
- added CN?: 2908-05WB-M6, MICROSD, symbol Adafruit VS1053 Headphone FeatherWing-eagle-import:MICROSD
- added D1, D2: WS2812B, LED_SMD:LED_WS2812B_PLCC4_5.0x5.0mm_P3.2mm, symbol LED:WS2812B
- added D?: MBR120, SOD-123, symbol Adafruit Feather M0 Basic rev C-eagle-import:DIODE-SCHOTTKYSOD-123
- added D?: LED, symbol Device:LED
- added FB? (x2): FERITTE, 0805-NO, symbol Adafruit VS1053 Headphone FeatherWing-eagle-import:FERRITE-0805NO
- added L?: RED, CHIPLED_0805_NOOUTLINE, symbol Adafruit Feather M0 Basic rev C-eagle-import:LED0805_NOOUTLINE
- added L?: 4.7μH, symbol pspice:INDUCTOR
- added R?: 2.2K, 0603-NO, symbol Adafruit Feather M0 Basic rev C-eagle-import:RESISTOR_0603_NOOUT
- added R?: 0.33, symbol Device:R
- added R?: 10K\, 0603-NO, symbol Adafruit Feather M0 Basic rev C-eagle-import:RESISTOR_0603_NOOUT
- added R? (x2): 100, 0603-NO, symbol Adafruit VS1053 Headphone FeatherWing-eagle-import:RESISTOR_0603_NOOUT
- added R?: 1M, 0603-NO, symbol Adafruit VS1053 Headphone FeatherWing-eagle-import:RESISTOR_0603_NOOUT
- added R?: 1K, 0603-NO, symbol Adafruit Feather M0 Basic rev C-eagle-import:RESISTOR_0603_NOOUT
- added R? (x2): 10K, 0805-NO, symbol Adafruit MPR121 Breakout-eagle-import:RESISTOR0805_NOOUTLINE
- added R?: 75K, 0805-NO, symbol Adafruit MPR121 Breakout-eagle-import:RESISTOR0805_NOOUTLINE
- added R? (x4): 100K, RESPACK_4X0603, symbol Adafruit VS1053 Headphone FeatherWing-eagle-import:RESISTOR_4PACK
- added R? (x2): 100k, 0603-NO, symbol Adafruit Feather M0 Basic rev C-eagle-import:RESISTOR_0603_NOOUT
- added R?: 100K, symbol Device:R
- added R? (x2): 22, 0603-NO, symbol Adafruit VS1053 Headphone FeatherWing-eagle-import:RESISTOR_0603_NOOUT
- added R?: 100K, 0603-NO, symbol Adafruit Feather M0 Basic rev C-eagle-import:RESISTOR_0603_NOOUT
- added R?: 100K, 0603-NO, symbol Adafruit VS1053 Headphone FeatherWing-eagle-import:RESISTOR_0603_NOOUT
- added SW?: SPST_TACT-KMR2, KMR2, symbol Adafruit Feather M0 Basic rev C-eagle-import:SPST_TACT-KMR2
- added TH?: 100k NTC, symbol Device:Thermistor_NTC
- added TP?: 3.3V, symbol Connector:TestPoint
- added TP?: BM83_USB_DP, symbol Connector:TestPoint
- added TP?: BM83_USB_DN, symbol Connector:TestPoint
- added TP?: 5V VBUS, symbol Connector:TestPoint
- added TP?: 1.8V, symbol Connector:TestPoint
- added TP?: BM83_LED2, symbol Connector:TestPoint
- added TP?: BM83_MFB, symbol Connector:TestPoint
- added TP?: GND, symbol Connector:TestPoint
- added TP?: BM83_LED1, symbol Connector:TestPoint
- added TP? (x2): TESTPOINTROUND1.5MM, TESTPOINT_ROUND_1.5MM, symbol Adafruit Feather M0 Basic rev C-eagle-import:TESTPOINTROUND1.5MM
- added U$?: ATSAMD21G18_QFN, TQFN48_7MM, symbol Adafruit Feather M0 Basic rev C-eagle-import:ATSAMD21J_QFN
- added U?: MCP73831T-2ACI/OT, SOT23-5, symbol Adafruit Feather M0 Basic rev C-eagle-import:MCP73831/2
- added U?: SPX3819-3.3, SOT23-5, symbol Adafruit Feather M0 Basic rev C-eagle-import:VREG_SOT23-5
- added U?: AP7312-1833W6-7, SOT23-6, symbol Adafruit VS1053 Headphone FeatherWing-eagle-import:VREG_SOT23-6_DUALAP7312
- added U?: MPR121Q, QFN20_3MM_NOTHERMAL, symbol Adafruit MPR121 Breakout-eagle-import:MPR121Q
- added U?: VS1053B, LQFP48, symbol Adafruit VS1053 Headphone FeatherWing-eagle-import:VS1053B
- added U?: MCP1643xMS, Package_SO:MSOP-8_3x3mm_P0.65mm, symbol Driver_LED:MCP1643xMS
- added X?: 32.768, XTAL3215, symbol Adafruit Feather M0 Basic rev C-eagle-import:XTAL-3.2X1.5
- added X?: JSTPH, JSTPH2, symbol Adafruit Feather M0 Basic rev C-eagle-import:CON_JST_PH_2PIN
- added X?: microUSB, 4UCONN_20329_V2, symbol Adafruit Feather M0 Basic rev C-eagle-import:USB_MICRO_20329_V2
- added Y?: ABM8G-12.288MHZ-4Y-T3, CRYSTAL_3.2X2.5, symbol Adafruit VS1053 Headphone FeatherWing-eagle-import:CRYSTAL3.2X2.5
Connections:
- net DN: now also TP?.1
- net DP: now also TP?.1
- net GND: now also C?.2, C?.2, C?.2, C?.2, C?.2, C?.2, C?.2, C?.2, C?.2, C?.2, C?.2, C?.2, C?.2, C?.2, C?.2, C?.2, C?.2, CN?.6 (GND@3), CN?.MT1 (GND@2), CN?.MT2 (GND@1), D1.3 (VSS), D2.3 (VSS), FB?.1 (P$1), L?.C, R?.1, R?.2, R?.2, R?.2, R?.2, R?.4 (1), R?.6 (2), SW?.2 (S), SW?.4 (S1), TP?.1, U$?.18 (GND), U$?.35 (GND), U$?.42 (GND), U$?.5 (GNDA), U$?.THERMAL (GND), U?.16 (DGND@1), U?.2 (GND), U?.2 (GND), U?.2 (VSS), U?.20 (DGND@2), U?.21 (DGND@3), U?.22 (DGND@4), U?.35 (GND), U?.4 (ADDR), U?.4 (DGND@0), U?.6 (PGND), U?.6 (VSS), U?.7 (SGND), X?.1, X?.BASE@1 (GND), X?.BASE@2 (GND), X?.GND, X?.SPRT@1 (GND), X?.SPRT@2 (GND), X?.SPRT@3 (GND), X?.SPRT@4 (GND)
- net LED1: now also TP?.1
- net LED2: now also TP?.1
- net PWR(MFB): now also TP?.1
- net ADAP_IN renamed +3V3
- net +3V3: now also C?.1, C?.1, C?.1, C?.1, D1.1 (VDD), D2.1 (VDD), R?.2, R?.2, TH?.1, TP?.1, U$?.17 (VDDIO), U$?.36 (VDDIO), U$?.44 (VDDIN), U$?.6 (VDDA), U?.3 (EN2), U?.4 (EN1), U?.5 (OUT), U?.5 (VIN)
- net P8_5 renamed BM83_UART_TX
- net BM83_UART_TX: now also U$?.16 (PA11/I11/AIN19/SERCOM0+2.3/I2SF0)
- net P8_6 renamed BM83_UART_RX
- net BM83_UART_RX: now also U$?.15 (PA10/I10/AIN18/SERCOM0+2.2/I2SCK)
- net RST_N renamed ~{RESET}
- net ~{RESET}: now also C?.1, R?.2, SW?.1 (P), SW?.3 (P1), U$?.40 (/RESET), U?.3 (XRESET)
- new net: L?.A, R?.2
- new net: D?.1 (K), R?.1, U?.2 (VFB)
- new net: D1.2 (DOUT), D2.4 (DIN)
- new net: R?.1, U?.5 (PROG)
- new net: CHG?.C, R?.1
- new net: C?.+, R?.1 (x2)
- new net: C?.1, R?.1, U?.17 (XTALOUT), Y?.1
- new net: C?.1, R?.2, U?.18 (XTALIN), Y?.2
- new net: R?.2, U?.1 (STAT)
- new net: R?.2, U?.7 (REXT)
- new net: C?.1, U?.5 (VREG)
- new net: L?.2, U?.5 (SW)
- new net: D?.2 (A), U?.4 (VOUT)
- new net: C?.1, U$?.1 (PA00/EINT0/SERCOM1.0), X?.P$1
- new net: C?.1, U$?.2 (PA01/EINT1/SERCOM1.1), X?.P$2
- new net: C?.1, U$?.43 (VDDCORE)
- new net: C?.1, R?.2 (x2)
- new net: C?.1, U?.44 (RCAP)
- new net 1.8V: C?.1, TP?.1, U?.24 (CVDD@2), U?.31 (CVDD@3), U?.5 (CVDD@0), U?.6 (VOUT1), U?.7 (CVDD@1)
- new net 3.3V: C?.1, C?.1, CN?.4 (SD_VDD), FB?.1 (P$1), R?.7 (2), R?.8 (2), U?.1 (VOUT2), U?.14 (IOVDD@1), U?.19 (IOVDD@2), U?.20 (VDD), U?.32 (XTEST), U?.6 (IOVDD@0)
- new net A0: U$?.3 (PA02/EINT2/AIN0/Y0/VOUT)
- new net A1: U$?.7 (PB08/I8/AIN2/SERCOM4.0)
- new net A2: U$?.8 (PB09/I9/AIN3/SERCOM4.1)
- new net A3: U$?.9 (PA04/EINT4/VREFB/AIN4/SERCOM0.0)
- new net A4: U$?.10 (PA05/EINT5/AIN5/SERCOM0.1)
- new net A5: R?.1, TH?.2, U$?.47 (PB02/I2/AIN10/SERCOM5.0)
- new net AGND: C?.2, C?.2, C?.2, C?.2, FB?.2 (P$2), U?.37 (AGND@0), U?.40 (AGND@1), U?.41 (AGND@2), U?.47 (AGND@3)
- new net AREF: C?.1, U$?.4 (PA03/EINT3/VREFA/AIN1)
- new net AVDD: C?.1, FB?.2 (P$2), R?.1, U?.38 (AVDD@0), U?.43 (AVDD@1), U?.45 (AVDD@2)
- new net CLKOUT: U?.15 (VCO)
- new net D+: U$?.34 (PA25/I13/SERCOM3+5.3/D+), X?.D+
- new net D-: U$?.33 (PA24/I12/SERCOM3+5.2/D-), X?.D-
- new net D10: U$?.27 (PA18/I2/SERCOM1+3.2), U?.13 (XDCS/BSYNC)
- new net D11: U$?.25 (PA16/I2C/I0/SERCOM1+3.0), U?.1 (EN)
- new net D12: U$?.28 (PA19/I3/SERCOM1+3.3/I2SD0), U?.1 (#IRQ)
- new net D13: R?.1, U$?.26 (PA17/I2C/I1/SERCOM1+3.1)
- new net D2: U$?.23 (PA14/I14/SERCOM2+4.2)
- new net D3: U$?.14 (PA09/I2C/I9/AIN17/SERCOM0+2.1/I2SMC)
- new net D4: U$?.13 (PA08/I2C/AIN16/SERCOM0+2.0/I2SD1)
- new net D5: CN?.2 (CS), R?.1, U$?.24 (PA15/I15/SERCOM3+4.3)
- new net D6: R?.2 (1), U$?.29 (PA20/I4/SERCOM3+5.2/I2SSC), U?.23 (XCS)
- new net D7: U$?.30 (PA21/I5/SERCOM3+5.3/I2SFS0)
- new net D8: U$?.11 (PA06/EINT6/AIN6/SERCOM0.2)
- new net D9: R?.1, R?.2, U$?.12 (PA07/I7/AIN7/SERCOM0.3/I2SD0), U?.8 (DREQ)
- new net ELEC0: U?.8 (ELE0)
- new net ELEC1: U?.9 (ELE1)
- new net ELEC10: U?.18 (ELE10/LED6)
- new net ELEC11: U?.19 (ELE11/LED7)
- new net ELEC2: U?.10 (ELE2)
- new net ELEC3: U?.11 (ELE3)
- new net ELEC4: U?.12 (ELE4/LED0)
- new net ELEC5: U?.13 (ELE5/LED1)
- new net ELEC6: U?.14 (ELE6/LED2)
- new net ELEC7: U?.15 (ELE7/LED3)
- new net ELEC8: U?.16 (ELE8/LED4)
- new net ELEC9: U?.17 (ELE9/LED5)
- new net EN: R?.2, U?.3 (EN)
- new net GPIO0: R?.5 (2), U?.33 (GPIO0)
- new net GPIO1: R?.3 (1), U?.34 (GPIO1)
- new net L_OUT: C?.-
- new net MISO: CN?.7 (DATA_OUT), U$?.21 (PA12/I12/I2C/SERCOM2+4.0), U?.30 (SO)
- new net MOSI: CN?.3 (DATA_IN), U$?.19 (PB10/I10/SERCOM4.2/I2SMC), U?.29 (SI)
- new net R_OUT: C?.-
- new net SCK: U$?.20 (PB11/I11/SERCOM4.3/I2SCL)
- new net SCL: R?.1, U$?.32 (PA23/I2C/I7/SERCOM3+5.1/SOF), U?.2 (SCL)
- new net SCLK: CN?.5 (SCLK), U?.28 (SCLK)
- new net SDA: R?.1, U$?.31 (PA22/I2C/I6/SERCOM3+5.0), U?.3 (SDA)
- new net SWCLK: TP?.P$1, U$?.45 (PA30/I10/SECOM1.2/SWCLK)
- new net SWDIO: TP?.P$1, U$?.46 (PA31/I11/SECOM1.3/SWDIO)
- new net VBAT: C?.1, D?.A, R?.1, U?.3 (VBAT), X?.2
- new net VBUS: C?.1, CHG?.A, D?.C, L?.1, R?.1, TP?.1, U?.1 (IN), U?.4 (VDD), U?.8 (VIN), X?.VBUS
- new net vs1053_LEFT: R?.1, R?.2, U?.46 (LEFT)
- new net vs1053_RIGHT: R?.1, R?.2, U?.39 (RIGHT)
Other:
- note added: "'clicks' ... this setup should minimize"
- note added: "1 / (2*π*f*Xc)"
- note added: "1 / (6.2832*20hz*16)"
- note added: "1 / (6.2832*20hz*32)"
- note added: "1.0K = 1000mA"
- note added: "10K = 100mA"
- note added: "16 ohm load at 20Hz cuttoff"
- note added: "1M resistor for DC bias"
- note added: "2.0K = 500mA"
- note added: "3.3v supply"
- note added: "32 ohm load at 20Hz cuttoff"
- note added: "5.0K = 200mA"
- note added: "= 249µF"
- note added: "= 497µF"
- note added: "Analog Supply Filtering"
- note added: "C1, C2 ="
- note added: "C4,C5 = 10pF"
- note added: "C4,C5 = 2*10pF - 2*5pF"
- note added: "C4,C5 = 2*CL - 2*Cstray"
- note added: "Caps: UKA0J471MPD1TD"
- note added: "DREQ high = at least 32 bytes"
- note added: "Disable SPI boot with GPIO0 low"
- note added: "Enabling the IC too soon can cause"
- note added: "N/C"
- note added: "POWER AND FILTERING"
- note added: "Power LED"
- note added: "RED LED"
- note added: "RESET"
- note added: "RGB LEDS"
- note added: "RXD"
- note added: "RXLED"
- note added: "SPI CS Pullups"
- note added: "TXD"
- note added: "TXLED"
- note added: "USB AND BATTERY CHARGING"
- note added: "USBHOSTEN"
- note added: "VS1053 oscillator requires"
- note added: "damage the earphones and causes"
- note added: "free in FIFO"
- note added: "http://www.vlsi.fi/uploads/media/vs10XXan.pdf"
- note added: "that. See section 8 of"
- note added: "transients during power up which can"
- note added: "vs1053 1.8v supply"
- moved on the sheet: U?

Commit message: main sch labelling 05 04 22
Parts:
- removed TP? (x2): TESTPOINTROUND1.5MM, TESTPOINT_ROUND_1.5MM, symbol Adafruit Feather M0 Basic rev C-eagle-import:TESTPOINTROUND1.5MM
- added J?: CAP TOUCH SLIDER, symbol Connector:Conn_01x12_Male
Connections:
- net ELEC0: now also J?.1 (Pin_1)
- net ELEC1: now also J?.2 (Pin_2)
- net ELEC10: now also J?.11 (Pin_11)
- net ELEC11: now also J?.12 (Pin_12)
- net ELEC2: now also J?.3 (Pin_3)
- net ELEC3: now also J?.4 (Pin_4)
- net ELEC4: now also J?.5 (Pin_5)
- net ELEC5: now also J?.6 (Pin_6)
- net ELEC6: now also J?.7 (Pin_7)
- net ELEC7: now also J?.8 (Pin_8)
- net ELEC8: now also J?.9 (Pin_9)
- net ELEC9: now also J?.10 (Pin_10)
Other:
- note added: "SAMD21 MCU"
- note added: "Touch Slider"
- note added: "VS1053B AUDIO CODEC"
- moved on the sheet: C?, CHG?, D?, FB?, R?, TP?, U?, X?

Commit message: main sch symbols 05 04 22
Parts:
- removed D2: WS2812B, LED_SMD:LED_WS2812B_PLCC4_5.0x5.0mm_P3.2mm, symbol LED:WS2812B
- removed D?: LED, symbol Device:LED
- removed L?: 4.7μH, symbol pspice:INDUCTOR
- removed R?: 0.33, symbol Device:R
- removed TP?: GND, symbol Connector:TestPoint
- removed U?: MCP1643xMS, Package_SO:MSOP-8_3x3mm_P0.65mm, symbol Driver_LED:MCP1643xMS
- added C50: 10µF, 0805-NO, symbol Adafruit Feather M0 Basic rev C-eagle-import:CAP_CERAMIC0805-NOOUTLINE
- added C600: (no value), symbol Adafruit Feather M0 Basic rev C-eagle-import:CAP_CERAMIC0603_NO
- added C601, C602, C603, C604, C605, C606, C607, C608, C609, C610, C611: 1uF, 0603-NO, symbol Adafruit Feather M0 Basic rev C-eagle-import:CAP_CERAMIC0603_NO
- added D50: LED, symbol Device:LED
- added D601, D602, D603, D604, D605, D606, D607, D608, D609, D610, D611: WS2812B, LED_SMD:LED_WS2812B_PLCC4_5.0x5.0mm_P3.2mm, symbol LED:WS2812B
- added L50: 4.7μH, symbol pspice:INDUCTOR
- added R50: (no value), symbol Device:R
- added TP73: GND, symbol Connector:TestPoint
- added U5: PAM2804, Package_TO_SOT_SMD:TSOT-23-5, symbol PAM2804:PAM2804
- C78: renamed from C?; value 10µF -> (none); footprint 0805-NO -> (none)
- U1: renamed from U$?; value ATSAMD21G18_QFN -> (none); footprint TQFN48_7MM -> (none)
- gave numbers to parts that had none: 63
- renumbered D1 to D600
Connections:
- net +3V3: now also U2.14 (IOVDD@1), U2.19 (IOVDD@2), U2.32 (XTEST), U2.6 (IOVDD@0), C600.1, C601.1, C602.1, C603.1, C604.1, C605.1, C606.1, C607.1, C608.1, C609.1, C610.1, C611.1, D601.1 (VDD), D602.1 (VDD), D603.1 (VDD), D604.1 (VDD), D605.1 (VDD), D606.1 (VDD), D607.1 (VDD), D608.1 (VDD), D609.1 (VDD), D610.1 (VDD), D611.1 (VDD)
- net 1.8V: no longer TP72.1
- net 3.3V: no longer U2.14 (IOVDD@1), U2.19 (IOVDD@2), U2.32 (XTEST), U2.6 (IOVDD@0)
- net A4: now also R74.2, R75.1
- net AGND: no longer C20.2, C80.2, C81.2, FB70.2 (P$2), U2.37 (AGND@0), U2.40 (AGND@1), U2.41 (AGND@2), U2.47 (AGND@3)
- net AVDD: no longer FB71.2 (P$2), R20.1, U2.38 (AVDD@0), U2.43 (AVDD@1), U2.45 (AVDD@2)
- net D11: now also U5.1 (EN)
- net D2: now also D600.4 (DIN)
- net D9: no longer R74.2, R75.1
- net GND: now also C50.2, C600.2, C601.2, C602.2, C603.2, C604.2, C605.2, C606.2, C607.2, C608.2, C609.2, C610.2, C611.2, D601.3 (VSS), D602.3 (VSS), D603.3 (VSS), D604.3 (VSS), D605.3 (VSS), D606.3 (VSS), D607.3 (VSS), D608.3 (VSS), D609.3 (VSS), D610.3 (VSS), D611.3 (VSS), R50.2, TP73.1, U5.2 (GND)
- net VBUS: now also U5.4 (VIN)
- net at D600.2 (DOUT): now also D601.4 (DIN)
- new net: D50.1 (K), R50.1, U5.5 (FB)
- new net: C50.1, D50.2 (A), L50.2
- new net: D607.2 (DOUT), D608.4 (DIN)
- new net: D606.2 (DOUT), D607.4 (DIN)
- new net: L50.1, U5.3 (SW)
- new net: D610.2 (DOUT), D611.4 (DIN)
- new net: D609.2 (DOUT), D610.4 (DIN)
- new net: D603.2 (DOUT), D604.4 (DIN)
- new net: D602.2 (DOUT), D603.4 (DIN)
- new net: D605.2 (DOUT), D606.4 (DIN)
- new net: D604.2 (DOUT), D605.4 (DIN)
- new net: D608.2 (DOUT), D609.4 (DIN)
- new net: D601.2 (DOUT), D602.4 (DIN)
- new net +1V8: TP72.1
- new net GNDA: C20.2, C80.2, C81.2, FB70.2 (P$2), U2.37 (AGND@0), U2.40 (AGND@1), U2.41 (AGND@2), U2.47 (AGND@3)
- new net VDDA: FB71.2 (P$2), R20.1, U2.38 (AVDD@0), U2.43 (AVDD@1), U2.45 (AVDD@2)
Other:
- note added: "AUDIO MUX (8)"
- note added: "BM83 BTM (3)"
- note added: "POWER AND FILTERING (7)"
- note added: "Power LED (5)"
- note added: "RGB LEDS (6)"
- note added: "SAMD21 MCU (1)"
- note added: "Touch Slider (4)"
- note added: "VS1053B AUDIO CODEC (2)"
- note removed: "POWER AND FILTERING"
- note removed: "Power LED"
- note removed: "RGB LEDS"
- note removed: "SAMD21 MCU"
- note removed: "Touch Slider"
- note removed: "VS1053B AUDIO CODEC"
- moved on the sheet: C20, C21, C22, C23, C24, C40, C41, C70, C71, C72, C73, C74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
