File: V2/electronics/main/main.kicad_sch (KiCad schematic)
At the start: 99 parts

Commit message: main sch footprints 07 04 22
Parts:
- C10, C20, C24, C600, C601, C602, C603, C604, C605, C606, C607, C608, C609, C610, C611, C70, C73, C76: value (none) -> 1uF; footprint (none) -> Capacitor_SMD:C_0603_1608Metric
- C12, C13, C22, C23: value (none) -> 22pF; footprint (none) -> Capacitor_SMD:C_0603_1608Metric
- C21: value (none) -> 0.1µF; footprint (none) -> Capacitor_SMD:C_0603_1608Metric
- C40, C41: value (none) -> 0.1uF; footprint (none) -> Capacitor_SMD:C_0603_1608Metric
- C50, C71, C72, C74, C75, C77, C78: value (none) -> 10uF; footprint (none) -> Capacitor_SMD:C_0805_2012Metric
- C80, C81: value (none) -> 10nF; footprint (none) -> Capacitor_SMD:C_0603_1608Metric
- C82, C83: value (none) -> 220uF; footprint (none) -> PANASONIC_C
- CHG1: value (none) -> ORANGE; footprint (none) -> CHIPLED_0805_NOOUTLINE
- CN20: value (none) -> 2908-05WB-M6; footprint (none) -> Connector_Card:microSD_HC_Hirose_DM3D-SF
- CN70: value (none) -> microUSB; footprint (none) -> 4UCONN_20329_V2
- CN71: value (none) -> JSTPH; footprint (none) -> Connector_JST:JST_PH_B2B-PH-SM4-TB_1x02-1MP_P2.00mm_Vertical
- D10: value (none) -> RED; footprint (none) -> LED_SMD:LED_0603_1608Metric
- D50: value (none) -> PWR_LED
- D600, D601, D602, D603, D604, D605, D606, D607, D608, D609, D610, D611: value (none) -> SK6812; footprint (none) -> LED_SMD:LED_SK6812_PLCC4_5.0x5.0mm_P3.2mm
- D71: value (none) -> MBR120; footprint (none) -> Diode_SMD:D_SOD-123
- FB70, FB71: value (none) -> FERITTE; footprint (none) -> Resistor_SMD:R_0805_2012Metric
- J40: value (none) -> CAP TOUCH SLIDER
- L50: value (none) -> 4.7μH
- R10: value (none) -> 2.2K; footprint (none) -> Resistor_SMD:R_0603_1608Metric
- R20, R75: value (none) -> 100K; footprint (none) -> Resistor_SMD:R_0603_1608Metric
- R21: value (none) -> 100K; footprint (none) -> Resistor_SMD:R_Array_Convex_4x0603
- R22: value (none) -> 1M; footprint (none) -> Resistor_SMD:R_0603_1608Metric
- R40: value (none) -> 75K; footprint (none) -> Resistor_SMD:R_0603_1608Metric
- R41, R42: value (none) -> 10K; footprint (none) -> Resistor_SMD:R_0603_1608Metric
- R50: value (none) -> 0.33
- R51: value (none) -> 100K
- R71, R74: value (none) -> 100k; footprint (none) -> Resistor_SMD:R_0603_1608Metric
- R72: value (none) -> 1K; footprint (none) -> Resistor_SMD:R_0603_1608Metric
- R73: value (none) -> 10K\; footprint (none) -> Resistor_SMD:R_0603_1608Metric
- R80, R81: value (none) -> 22; footprint (none) -> Resistor_SMD:R_0603_1608Metric
- R82, R83: value (none) -> 100; footprint (none) -> Resistor_SMD:R_0603_1608Metric
- SW1: value (none) -> SPST_TACT-KMR2; footprint (none) -> Button_Switch_SMD:SW_Push_1P1T_NO_CK_KMR2
- TH50: value (none) -> 100k NTC
- TP30: value (none) -> BM83_MFB
- TP31: value (none) -> BM83_LED1
- TP32: value (none) -> BM83_LED2
- TP33: value (none) -> BM83_USB_DN
- TP34: value (none) -> BM83_USB_DP
- TP70: value (none) -> 5V VBUS
- TP71: value (none) -> 3.3V
- TP72: value (none) -> 1.8V
- TP73: value (none) -> GND
- U1: value (none) -> ATSAMD21G18_QFN; footprint (none) -> Package_DFN_QFN:TQFN-48-1EP_7x7mm_P0.5mm_EP5.1x5.1mm
- U2: value (none) -> VS1053B; footprint (none) -> Package_QFP:LQFP-48_7x7mm_P0.5mm
- U3: value (none) -> BM83; footprint (none) -> BM83:BM83
- U4: value (none) -> MPR121Q; footprint (none) -> Package_DFN_QFN:UQFN-20_3x3mm_P0.4mm
- U5: value (none) -> PAM2804; footprint (none) -> Package_TO_SOT_SMD:TSOT-23-5
- U6: value (none) -> AP22814AW5; footprint (none) -> Package_TO_SOT_SMD:SOT-23-5
- U70: value (none) -> SPX3819-3.3; footprint (none) -> Package_TO_SOT_SMD:SOT-23-5
- U71: value (none) -> AP7312-1833W6-7; footprint (none) -> Package_TO_SOT_SMD:SOT-23-6
- U72: value (none) -> MCP73831T-2ACI/OT; footprint (none) -> Package_TO_SOT_SMD:SOT-23-5
- X10: value (none) -> 32.768; footprint (none) -> other footprints:XTAL3215
- X20: value (none) -> ABM8G-12.288MHZ-4Y-T3; footprint (none) -> other footprints:CRYSTAL_3.2X2.5

Commit message: main sch footprints 07 04 22
Parts:
- R50: value 0.33 -> (none)
- R51: value 100K -> (none)
Connections:
- net D8 is gone; now on net CHRG_STAT: U1.11 (PA06/EINT6/AIN6/SERCOM0.2)
- net +3V3: now also R72.1
- net VBUS: no longer CHG1.A
- net at CHG1.C: now also U72.1 (STAT); no longer R72.1
- net CHRG_STAT: now reaches R72.2
- net CHRG_STAT: now also CHG1.A; no longer U72.1 (STAT)
Other:
- moved on the sheet: CHG1, R72
Changed lines of the file:
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@@
   (junction (at 43.815 321.31) (diameter 0) (color 0 0 0 0)
   )
-  (junction (at 53.34 131.445) (diameter 0) (color 0 0 0 0)
-  )
   (junction (at 66.04 321.31) (diameter 0) (color 0 0 0 0)
   )
@@
     (stroke (width 0) (type default) (color 0 0 0 0))
   )
-  (wire (pts (xy 327.66 223.52) (xy 345.44 223.52))
+  (wire (pts (xy 327.66 223.52) (xy 389.89 223.52))
     (stroke (width 0) (type default) (color 0 0 0 0))
   )
@@
     (stroke (width 0) (type default) (color 0 0 0 0))
   )
-  (wire (pts (xy 45.72 131.445) (xy 53.34 131.445))
-    (stroke (width 0) (type default) (color 0 0 0 0))
-  )
   (wire (pts (xy 317.5 90.17) (xy 317.5 92.71))
     (stroke (width 0) (type default) (color 0 0 0 0))
@@
     (stroke (width 0) (type default) (color 0 0 0 0))
   )
+  (wire (pts (xy 389.89 227.33) (xy 389.89 223.52))
+    (stroke (width 0) (type default) (color 0 0 0 0))
+  )
   (wire (pts (xy 177.8 94.615) (xy 177.8 89.535))
     (stroke (width 0) (type default) (color 0 0 0 0))
@@
     (stroke (width 0) (type default) (color 0 0 0 0))
   )
-  (wire (pts (xy 389.89 227.33) (xy 389.89 222.25))
-    (stroke (width 0) (type default) (color 0 0 0 0))
-  )
   (wire (pts (xy 35.56 321.31) (xy 43.815 321.31))
     (stroke (width 0) (type default) (color 0 0 0 0))
@@
     (stroke (width 0) (type default) (color 0 0 0 0))
   )
-  (wire (pts (xy 76.2 136.525) (xy 81.28 136.525))
+  (wire (pts (xy 76.835 136.525) (xy 81.28 136.525))
     (stroke (width 0) (type default) (color 0 0 0 0))
   )
-  (wire (pts (xy 53.34 131.445) (xy 81.28 131.445))
+  (wire (pts (xy 45.72 131.445) (xy 81.28 131.445))
     (stroke (width 0) (type default) (color 0 0 0 0))
   )
@@
     (stroke (width 0) (type default) (color 0 0 0 0))
   )
-  (wire (pts (xy 53.34 136.525) (xy 53.34 131.445))
+  (wire (pts (xy 206.375 344.17) (xy 206.375 347.98))
     (stroke (width 0) (type default) (color 0 0 0 0))
   )
-  (wire (pts (xy 206.375 344.17) (xy 206.375 347.98))
+  (wire (pts (xy 60.325 136.525) (xy 69.215 136.525))
     (stroke (width 0) (type default) (color 0 0 0 0))
   )
@@
     (stroke (width 0) (type default) (color 0 0 0 0))
   )
+  (wire (pts (xy 45.72 136.525) (xy 50.165 136.525))
+    (stroke (width 0) (type default) (color 0 0 0 0))
+  )
   (wire (pts (xy 88.265 277.495) (xy 88.265 287.655))
     (stroke (width 0) (type default) (color 0 0 0 0))
@@
     (stroke (width 0) (type default) (color 0 0 0 0))
   )
-  (wire (pts (xy 55.88 136.525) (xy 53.34 136.525))
-    (stroke (width 0) (type default) (color 0 0 0 0))
-  )
   (wire (pts (xy 104.775 179.07) (xy 120.015 179.07))
     (stroke (width 0) (type default) (color 0 0 0 0))
@@
     (stroke (width 0) (type default) (color 0 0 0 0))
   )
-  (wire (pts (xy 63.5 136.525) (xy 66.04 136.525))
-    (stroke (width 0) (type default) (color 0 0 0 0))
-  )
   (wire (pts (xy 529.59 220.345) (xy 547.37 220.345))
     (stroke (width 0) (type default) (color 0 0 0 0))
@@
     (effects (font (size 1.2446 1.2446)) (justify right bottom))
   )
-  (label "D13" (at 389.89 222.25 270)
-    (effects (font (size 1.2446 1.2446)) (justify right bottom))
-  )
   (label "RGB_VDD" (at 88.265 234.315 0)
     (effects (font (size 1.27 1.27)) (justify left bottom))
@@
     (effects (font (size 1.2446 1.2446)) (justify left bottom))
   )
+  (label "CHRG_STAT" (at 345.44 190.5 0)
+    (effects (font (size 1.27 1.27)) (justify left bottom))
+  )
   (label "RGB_VDD" (at 110.49 234.315 0)
     (effects (font (size 1.27 1.27)) (justify left bottom))
@@
     (effects (font (size 1.2446 1.2446)) (justify left bottom))
   )
+  (label "CHRG_STAT" (at 60.325 136.525 0)
+    (effects (font (size 1.27 1.27)) (justify left bottom))
+  )
   (label "vs1053_LEFT" (at 494.665 220.345 0)
     (effects (font (size 1.2446 1.2446)) (justify left bottom))
@@
     (pin "1")
   )
-  (symbol (lib_id "Adafruit Feather M0 Basic rev C-eagle-import:LED0805_NOOUTLINE") (at 60.96 136.525 0) (unit 1)
+  (symbol (lib_id "Adafruit Feather M0 Basic rev C-eagle-import:LED0805_NOOUTLINE") (at 74.295 136.525 0) (unit 1)
     (in_bom yes) (on_board yes)
-    (property "Reference" "CHG1" (id 0) (at 59.69 132.08 0))
-    (property "Value" "ORANGE" (id 1) (at 59.69 139.319 0))
-    (property "Footprint" "CHIPLED_0805_NOOUTLINE" (id 2) (at 60.96 136.525 0)
+    (property "Reference" "CHG1" (id 0) (at 73.025 132.08 0))
+    (property "Value" "ORANGE" (id 1) (at 73.025 139.319 0))
+    (property "Footprint" "CHIPLED_0805_NOOUTLINE" (id 2) (at 74.295 136.525 0)
       (effects (font (size 1.27 1.27)) hide)
     )
-    (property "Datasheet" "" (id 3) (at 60.96 136.525 0)
+    (property "Datasheet" "" (id 3) (at 74.295 136.525 0)
       (effects (font (size 1.27 1.27)) hide)
     )
@@
     (pin "2")
   )
-  (symbol (lib_id "Adafruit Feather M0 Basic rev C-eagle-import:RESISTOR_0603_NOOUT") (at 71.12 136.525 0) (unit 1)
+  (symbol (lib_id "Adafruit Feather M0 Basic rev C-eagle-import:RESISTOR_0603_NOOUT") (at 55.245 136.525 0) (unit 1)
     (in_bom yes) (on_board yes)
-    (property "Reference" "R72" (id 0) (at 71.12 133.985 0))
-    (property "Value" "1K" (id 1) (at 71.12 136.525 0)
+    (property "Reference" "R72" (id 0) (at 55.245 133.985 0))
+    (property "Value" "1K" (id 1) (at 55.245 136.525 0)
       (effects (font (size 1.016 1.016) bold))
     )
-    (property "Footprint" "Resistor_SMD:R_0603_1608Metric" (id 2) (at 71.12 136.525 0)
+    (property "Footprint" "Resistor_SMD:R_0603_1608Metric" (id 2) (at 55.245 136.525 0)
       (effects (font (size 1.27 1.27)) hide)
     )
-    (property "Datasheet" "" (id 3) (at 71.12 136.525 0)
+    (property "Datasheet" "" (id 3) (at 55.245 136.525 0)
       (effects (font (size 1.27 1.27)) hide)
     )
@@
     (pin "1")
     (pin "8")
+    (pin "2")
+    (pin "7")
+    (pin "3")
+    (pin "6")
+    (pin "4")
+    (pin "5")
   )
   (symbol (lib_id "Adafruit VS1053 Headphone FeatherWing-eagle-import:RESISTOR_4PACK") (at 241.3 117.475 0) (unit 4)
@@
       (effects (font (size 1.27 1.27)) hide)
     )
+    (pin "1")
+    (pin "8")
+    (pin "2")
+    (pin "7")
+    (pin "3")
+    (pin "6")
     (pin "4")
     (pin "5")
@@
       (effects (font (size 1.27 1.27)) (justify left))
     )
-    (property "Value" "100K" (id 1) (at 219.71 342.2649 0)
+    (property "Value" "" (id 1) (at 219.71 342.2649 0)
       (effects (font (size 1.27 1.27)) (justify left))
     )
@@
       (effects (font (size 1.27 1.27)) hide)
     )
+    (pin "1")
+    (pin "8")
+    (pin "2")
+    (pin "7")
     (pin "3")
     (pin "6")
+    (pin "4")
+    (pin "5")
   )
   (symbol (lib_id "power:+3V3") (at 318.135 302.26 0) (unit 1)
@@
       (effects (font (size 1.27 1.27)) (justify left))
     )
-    (property "Value" "0.33" (id 1) (at 192.913 342.8616 0)
+    (property "Value" "" (id 1) (at 192.913 342.8616 0)
       (effects (font (size 1.27 1.27)) (justify left))
     )
@@
       (effects (font (size 1.27 1.27)) hide)
     )
+    (pin "1")
+    (pin "8")
     (pin "2")
     (pin "7")
+    (pin "3")
+    (pin "6")
+    (pin "4")
+    (pin "5")
   )
   (symbol (lib_id "power:GND") (at 47.625 94.615 0) (unit 1)
@@
     (pin "1")
   )
+  (symbol (lib_id "power:+3V3") (at 45.72 136.525 90) (unit 1)
+    (in_bom yes) (on_board yes) (fields_autoplaced)
+    (property "Reference" "#PWR?" (id 0) (at 49.53 136.525 0)
+      (effects (font (size 1.27 1.27)) hide)
+    )
+    (property "Value" "" (id 1) (at 41.91 136.5249 90)
+      (effects (font (size 1.27 1.27)) (justify left))
+    )
+    (property "Footprint" "" (id 2) (at 45.72 136.525 0)
+      (effects (font (size 1.27 1.27)) hide)
+    )
+    (property "Datasheet" "" (id 3) (at 45.72 136.525 0)
+      (effects (font (size 1.27 1.27)) hide)
+    )
+    (pin "1")
+  )
   (symbol (lib_id "power:VDDA") (at 314.96 49.53 0) (unit 1)
     (in_bom yes) (on_board yes) (fields_autoplaced)
@@
       (reference "#PWR0199") (unit 1) (value "GNDA") (footprint "")
     )
+    (path "/f047a2e0-676e-4df9-b2ad-cd00cc8472b8"
+      (reference "#PWR?") (unit 1) (value "+3V3") (footprint "")
+    )
     (path "/fbe0d58b-5b0f-497e-9342-52d354ef51fe"
       (reference "#U$0101") (unit 1) (value "GND") (footprint "")
@@
     )
     (path "/7fe142c2-dd61-4d4c-80a4-311b9dc625d3"
-      (reference "R50") (unit 1) (value "0.33") (footprint "")
+      (reference "R50") (unit 1) (value "0.33") (footprint "Resistor_SMD:R_0603_1608Metric")
     )
     (path "/7a3cd876-ff7c-4e39-94dc-e7c5f10b931b"
-      (reference "R51") (unit 1) (value "100K") (footprint "")
+      (reference "R51") (unit 1) (value "100K") (footprint "Resistor_SMD:R_0603_1608Metric")
     )
     (path "/628370d6-13de-4e7a-8c74-1e79dd7bc426"

Commit message: main sch audio out tests 07 04 22
Parts:
- added C? (x2): 10nF, Capacitor_SMD:C_0603_1608Metric, symbol Adafruit VS1053 Headphone FeatherWing-eagle-import:CAP_CERAMIC0603_NO
- added C? (x2): 220uF, PANASONIC_C, symbol Adafruit VS1053 Headphone FeatherWing-eagle-import:CPOL-USC
- added R23: 100K, Resistor_SMD:R_0603_1608Metric, symbol Adafruit VS1053 Headphone FeatherWing-eagle-import:RESISTOR_0603_NOOUT
- added R? (x2): 22, Resistor_SMD:R_0603_1608Metric, symbol Adafruit VS1053 Headphone FeatherWing-eagle-import:RESISTOR_0603_NOOUT
- added R? (x2): 100, Resistor_SMD:R_0603_1608Metric, symbol Adafruit VS1053 Headphone FeatherWing-eagle-import:RESISTOR_0603_NOOUT
- R50: value (none) -> 0.33; footprint (none) -> Resistor_SMD:R_0603_1608Metric
- R51: value (none) -> 100K; footprint (none) -> Resistor_SMD:R_0603_1608Metric
Connections:
- net +3V3: no longer C24.1, CN20.4 (SD_VDD), FB71.1 (P$1), U2.14 (IOVDD@1), U2.19 (IOVDD@2), U2.32 (XTEST), U2.6 (IOVDD@0), U71.1 (VOUT2), U71.3 (EN2), U71.4 (EN1)
- net AOHPL: now also R?.1, R?.2
- net AOHPR: now also R?.1, R?.2
- net D4: now also U71.3 (EN2), U71.4 (EN1)
- net GNDA: now also C?.2, C?.2
- net L_OUT: now also C?.-
- net R_OUT: now also C?.-
- net at U2.26 (RX): now also R23.1
- new net: C?.1, R?.2 (x2)
- new net: C?.+, R?.1 (x2)
- new net +3.3VA: C24.1, CN20.4 (SD_VDD), FB71.1 (P$1), R23.2, U2.14 (IOVDD@1), U2.19 (IOVDD@2), U2.32 (XTEST), U2.6 (IOVDD@0), U71.1 (VOUT2)
Other:
- moved on the sheet: C74

Commit message: main sch footprints 08 04 22
Parts:
- C10, C20, C24, C600, C601, C602, C603, C604, C605, C606, C607, C608, C609, C610, C611, C70, C73, C76: value 1uF -> (none); footprint Capacitor_SMD:C_0603_1608Metric -> (none)
- C12, C13, C22, C23: value 22pF -> (none); footprint Capacitor_SMD:C_0603_1608Metric -> (none)
- C21: value 0.1µF -> (none); footprint Capacitor_SMD:C_0603_1608Metric -> (none)
- C40, C41: value 0.1uF -> (none); footprint Capacitor_SMD:C_0603_1608Metric -> (none)
- C50, C71, C72, C74, C75, C77, C78: value 10uF -> (none); footprint Capacitor_SMD:C_0805_2012Metric -> (none)
- C80, C81, C? (x2): value 10nF -> (none); footprint Capacitor_SMD:C_0603_1608Metric -> (none)
- C82, C83, C? (x2): value 220uF -> (none); footprint PANASONIC_C -> (none)
- CHG1: value ORANGE -> (none); footprint CHIPLED_0805_NOOUTLINE -> (none)
- CN20: value 2908-05WB-M6 -> (none); footprint Connector_Card:microSD_HC_Hirose_DM3D-SF -> (none)
- CN70: value microUSB -> (none); footprint 4UCONN_20329_V2 -> (none)
- CN71: value JSTPH -> (none); footprint Connector_JST:JST_PH_B2B-PH-SM4-TB_1x02-1MP_P2.00mm_Vertical -> (none)
- D10: value RED -> (none); footprint LED_SMD:LED_0603_1608Metric -> (none)
- D50: value PWR_LED -> (none)
- D600, D601, D602, D603, D604, D605, D606, D607, D608, D609, D610, D611: value SK6812 -> (none); footprint LED_SMD:LED_SK6812_PLCC4_5.0x5.0mm_P3.2mm -> (none)
- D71: value MBR120 -> (none); footprint Diode_SMD:D_SOD-123 -> (none)
- FB70, FB71: value FERITTE -> (none); footprint Resistor_SMD:R_0805_2012Metric -> (none)
- J40: value CAP TOUCH SLIDER -> (none)
- L50: value 4.7μH -> (none)
- R10: value 2.2K -> (none); footprint Resistor_SMD:R_0603_1608Metric -> (none)
- R20, R23, R51, R75: value 100K -> (none); footprint Resistor_SMD:R_0603_1608Metric -> (none)
- R21: value 100K -> (none); footprint Resistor_SMD:R_Array_Convex_4x0603 -> (none)
- R22: value 1M -> (none); footprint Resistor_SMD:R_0603_1608Metric -> (none)
- R40: value 75K -> (none); footprint Resistor_SMD:R_0603_1608Metric -> (none)
- R41, R42: value 10K -> (none); footprint Resistor_SMD:R_0603_1608Metric -> (none)
- R50: value 0.33 -> (none); footprint Resistor_SMD:R_0603_1608Metric -> (none)
- R71, R74: value 100k -> (none); footprint Resistor_SMD:R_0603_1608Metric -> (none)
- R72: value 1K -> (none); footprint Resistor_SMD:R_0603_1608Metric -> (none)
- R73: value 10K\ -> (none); footprint Resistor_SMD:R_0603_1608Metric -> (none)
- R80, R81, R? (x2): value 22 -> (none); footprint Resistor_SMD:R_0603_1608Metric -> (none)
- R82, R83, R? (x2): value 100 -> (none); footprint Resistor_SMD:R_0603_1608Metric -> (none)
- SW1: value SPST_TACT-KMR2 -> (none); footprint Button_Switch_SMD:SW_Push_1P1T_NO_CK_KMR2 -> (none)
- TH50: value 100k NTC -> (none)
- TP30: value BM83_MFB -> (none)
- TP31: value BM83_LED1 -> (none)
- TP32: value BM83_LED2 -> (none)
- TP33: value BM83_USB_DN -> (none)
- TP34: value BM83_USB_DP -> (none)
- TP70: value 5V VBUS -> (none)
- TP71: value 3.3V -> (none)
- TP72: value 1.8V -> (none)
- TP73: value GND -> (none)
- U1: value ATSAMD21G18_QFN -> (none); footprint Package_DFN_QFN:TQFN-48-1EP_7x7mm_P0.5mm_EP5.1x5.1mm -> (none)
- U2: value VS1053B -> (none); footprint Package_QFP:LQFP-48_7x7mm_P0.5mm -> (none)
- U3: value BM83 -> (none); footprint BM83:BM83 -> (none)
- U4: value MPR121Q -> (none); footprint Package_DFN_QFN:UQFN-20_3x3mm_P0.4mm -> (none)
- U5: value PAM2804 -> (none); footprint Package_TO_SOT_SMD:TSOT-23-5 -> (none)
- U6: value AP22814AW5 -> (none); footprint Package_TO_SOT_SMD:SOT-23-5 -> (none)
- U70: value SPX3819-3.3 -> (none); footprint Package_TO_SOT_SMD:SOT-23-5 -> (none)
- U71: value AP7312-1833W6-7 -> (none); footprint Package_TO_SOT_SMD:SOT-23-6 -> (none)
- U72: value MCP73831T-2ACI/OT -> (none); footprint Package_TO_SOT_SMD:SOT-23-5 -> (none)
- X10: value 32.768 -> (none); footprint other footprints:XTAL3215 -> (none)
- X20: value ABM8G-12.288MHZ-4Y-T3 -> (none); footprint other footprints:CRYSTAL_3.2X2.5 -> (none)
