File: V2/electronics/main/main.kicad_sch (KiCad schematic)
At the start: 108 parts

Commit message: pcb design done 24 04 22
Parts:
- removed C77: (no value), symbol Adafruit Feather M0 Basic rev C-eagle-import:CAP_CERAMIC0805-NOOUTLINE
- removed C82, C83, C? (x2): (no value), symbol Adafruit VS1053 Headphone FeatherWing-eagle-import:CPOL-USC
- removed CN71: (no value), symbol Adafruit Feather M0 Basic rev C-eagle-import:CON_JST_PH_2PIN
- removed R21: (no value), symbol Adafruit VS1053 Headphone FeatherWing-eagle-import:RESISTOR_4PACK
- removed R71: (no value), symbol Adafruit Feather M0 Basic rev C-eagle-import:RESISTOR_0603_NOOUT
- added C30, C51, C90: 10uF, Capacitor_SMD:C_0402_1005Metric, symbol Adafruit Feather M0 Basic rev C-eagle-import:CAP_CERAMIC0805-NOOUTLINE
- added C810, C82, C83, C86, C87, C88, C89: 1uf, Capacitor_SMD:C_0402_1005Metric, symbol Adafruit VS1053 Headphone FeatherWing-eagle-import:CAP_CERAMIC0603_NO
- added C91: 0.1uF, Capacitor_SMD:C_0402_1005Metric, symbol Adafruit Feather M0 Basic rev C-eagle-import:CAP_CERAMIC0805-NOOUTLINE
- added D72: MBR120, Diode_SMD:D_SOD-123, symbol Adafruit Feather M0 Basic rev C-eagle-import:DIODE-SCHOTTKYSOD-123
- added J10: Conn_01x20_Female, Connector_Hirose:Hirose_DF12_DF12E3.0-20DP-0.5V_2x10_P0.50mm_Vertical, symbol Connector:Conn_01x20_Female
- added J11: Conn_01x20_Male, Connector_Hirose:Hirose_DF12_DF12C3.0-20DS-0.5V_2x10_P0.50mm_Vertical, symbol Connector:Conn_01x20_Male
- added J5: Conn_01x05_Female, Connector_Hirose:Hirose_DF52-5S-0.8H_1x05-1MP_P0.80mm_Horizontal, symbol Connector:Conn_01x05_Female
- added J80: Conn_01x04_Female, Connector_Hirose:Hirose_DF52-5S-0.8H_1x05-1MP_P0.80mm_Horizontal, symbol Connector:Conn_01x05_Female
- added J81: Conn_01x02_Female, Connector_Hirose:Hirose_DF52-5S-0.8H_1x05-1MP_P0.80mm_Horizontal, symbol Connector:Conn_01x05_Female
- added R23, R24, R25, R26: 100K, Resistor_SMD:R_0402_1005Metric, symbol Adafruit VS1053 Headphone FeatherWing-eagle-import:RESISTOR_0603_NOOUT
- added R60: 470, Resistor_SMD:R_0402_1005Metric, symbol Adafruit Feather M0 Basic rev C-eagle-import:RESISTOR_0603_NOOUT
- added U8: max9725aetc+, footprints:max9725aetc&plus_, symbol 2022-04-11_15-45-50:max9725aetc+
- added U9: MP34DT01TR-M, PDM footprints:MP34DT01TR-M, symbol 2022-04-17_20-44-18:MP34DT01TR-M
- C10, C20, C24, C600, C601, C602, C603, C604, C605, C606, C607, C608, C609, C610, C611, C70, C76: value (none) -> 1uF; footprint (none) -> Capacitor_SMD:C_0402_1005Metric
- C11: renamed from C73; value (none) -> 1uF; footprint (none) -> Capacitor_SMD:C_0402_1005Metric
- C12, C13, C22, C23: value (none) -> 22pF; footprint (none) -> Capacitor_SMD:C_0402_1005Metric
- C21: value (none) -> 0.1µF; footprint (none) -> Capacitor_SMD:C_0402_1005Metric
- C40, C41: value (none) -> 0.1uF; footprint (none) -> Capacitor_SMD:C_0402_1005Metric
- C50, C71, C72, C74, C75: value (none) -> 10uF; footprint (none) -> Capacitor_SMD:C_0402_1005Metric
- C77: renamed from C78; value (none) -> 10uF; footprint (none) -> Capacitor_SMD:C_0402_1005Metric
- C80, C81: value (none) -> 10nF; footprint (none) -> Capacitor_SMD:C_0402_1005Metric
- C84, C85: renamed from C?; value (none) -> 10nF; footprint (none) -> Capacitor_SMD:C_0402_1005Metric
- CHG1: value (none) -> ORANGE; footprint (none) -> LED_SMD:LED_0603_1608Metric
- CN20: value (none) -> 2908-05WB-M6; footprint (none) -> Connector_Card:microSD_HC_Hirose_DM3D-SF
- CN70: value (none) -> microUSB; footprint (none) -> Connector_USB:USB_Micro-B_Molex-105017-0001
- D10: value (none) -> RED; footprint (none) -> LED_SMD:LED_0603_1608Metric
- D50: value (none) -> PWR_LED
- D600, D601, D602, D603, D604, D605, D606, D607, D608, D609, D610, D611: value (none) -> SK6812; footprint (none) -> LED_SMD:LED_SK6812_EC15_1.5x1.5mm
- D71: value (none) -> MBR120; footprint (none) -> Diode_SMD:D_SOD-123
- FB70, FB71: value (none) -> FERITTE; footprint (none) -> Resistor_SMD:R_0805_2012Metric
- J40: value (none) -> CAP TOUCH SLIDER
- L50: value (none) -> 4.7μH; footprint (none) -> Inductor_SMD:L_1210_3225Metric
- R10: value (none) -> 2.2K; footprint (none) -> Resistor_SMD:R_0402_1005Metric
- R20, R51: value (none) -> 100K; footprint (none) -> Resistor_SMD:R_0402_1005Metric
- R21: renamed from R23; value (none) -> 100K; footprint (none) -> Resistor_SMD:R_0402_1005Metric
- R22: value (none) -> 1M; footprint (none) -> Resistor_SMD:R_0402_1005Metric
- R40: value (none) -> 75K; footprint (none) -> Resistor_SMD:R_0402_1005Metric
- R41, R42, R73: value (none) -> 10K; footprint (none) -> Resistor_SMD:R_0402_1005Metric
- R50: value (none) -> 0.33; footprint (none) -> Resistor_SMD:R_0402_1005Metric
- R70: renamed from R75; value (none) -> 100K; footprint (none) -> Resistor_SMD:R_0402_1005Metric
- R71: renamed from R74; value (none) -> 100k; footprint (none) -> Resistor_SMD:R_0402_1005Metric
- R72: value (none) -> 1K; footprint (none) -> Resistor_SMD:R_0402_1005Metric
- R80, R81: value (none) -> 22; footprint (none) -> Resistor_SMD:R_0402_1005Metric
- R82, R83: value (none) -> 100; footprint (none) -> Resistor_SMD:R_0402_1005Metric
- R84, R85: renamed from R?; value (none) -> 22; footprint (none) -> Resistor_SMD:R_0402_1005Metric
- R86, R87: renamed from R?; value (none) -> 100; footprint (none) -> Resistor_SMD:R_0402_1005Metric
- SW1: value (none) -> SPST_TACT-KMR2; footprint (none) -> Button_Switch_SMD:SW_Push_1P1T_NO_CK_KMR2
- TH50: value (none) -> 100k NTC
- TP30: value (none) -> BM83_MFB; footprint (none) -> TestPoint:TestPoint_Pad_D1.0mm
- TP31: value (none) -> BM83_LED1; footprint (none) -> TestPoint:TestPoint_Pad_D1.0mm
- TP32: value (none) -> BM83_LED2; footprint (none) -> TestPoint:TestPoint_Pad_D1.0mm
- TP33: value (none) -> BM83_USB_DN; footprint (none) -> TestPoint:TestPoint_Pad_D1.0mm
- TP34: value (none) -> BM83_USB_DP; footprint (none) -> TestPoint:TestPoint_Pad_D1.0mm
- TP70: value (none) -> 5V VBUS; footprint (none) -> TestPoint:TestPoint_Pad_D1.0mm
- TP71: value (none) -> 3.3V; footprint (none) -> TestPoint:TestPoint_Pad_D1.0mm
- TP72: value (none) -> 1.8V; footprint (none) -> TestPoint:TestPoint_Pad_D1.0mm
- TP73: value (none) -> GND; footprint (none) -> TestPoint:TestPoint_Pad_D1.0mm
- U1: value (none) -> ATSAMD21G18_QFN; footprint (none) -> Package_DFN_QFN:TQFN-48-1EP_7x7mm_P0.5mm_EP5.1x5.1mm
- U2: value (none) -> VS1053B; footprint (none) -> Package_QFP:LQFP-48_7x7mm_P0.5mm
- U3: value (none) -> BM83; footprint (none) -> BM83:BM83
- U4: value (none) -> MPR121Q; footprint (none) -> Package_DFN_QFN:UQFN-20_3x3mm_P0.4mm
- U5: value (none) -> PAM2804; footprint (none) -> Package_TO_SOT_SMD:TSOT-23-5
- U6: value (none) -> AP22814AW5; footprint (none) -> Package_TO_SOT_SMD:SOT-23-5
- U70: value (none) -> SPX3819-3.3; footprint (none) -> Package_TO_SOT_SMD:SOT-23-5
- U71: value (none) -> AP7312-1833W6-7; footprint (none) -> Package_TO_SOT_SMD:SOT-23-6
- U72: value (none) -> MCP73831T-2ACI/OT; footprint (none) -> Package_TO_SOT_SMD:SOT-23-5
- X10: value (none) -> 32.768; footprint (none) -> other footprints:XTAL3215
- X20: value (none) -> ABM8G-12.288MHZ-4Y-T3; footprint (none) -> other footprints:CRYSTAL_3.2X2.5
Connections:
- net 1.8V is gone; now on net +1V8: U2.24 (CVDD@2)
- net EN is gone; now on net VBUS: U70.3 (EN)
- net SCK is gone; now on net SCLK: U1.20 (PB11/I11/SERCOM4.3/I2SCL)
- net +1V8: now also C810.1, J10.11 (Pin_11), J11.11 (Pin_11), U8.12 (~{SHDN}), U8.9 (VDD)
- net +3.3VA: now also R23.1, R24.1
- net +3V3: now also R20.1, U71.4 (EN1), C90.1, C91.1, J10.15 (Pin_15), J11.15 (Pin_15), J5.4 (Pin_4), U9.1 (VDD), U9.2 (LR); no longer U3.22 (ADAP_IN)
- net +BATT: now also D71.2 (A), J10.7 (Pin_7), J10.8 (Pin_8), J11.7 (Pin_7), J11.8 (Pin_8), J80.2 (Pin_2); no longer D71.A
- net A3: now also R51.1, TH50.2, J10.16 (Pin_16), J11.16 (Pin_16), J5.5 (Pin_5)
- net A5: no longer R51.1, TH50.2
- net AOHPL: now also R84.1, R86.2, J10.3 (Pin_3), J11.3 (Pin_3); no longer R85.1, R87.2
- net AOHPR: now also R85.1, R87.2, J10.4 (Pin_4), J11.4 (Pin_4); no longer R84.1, R86.2
- net CHRG_STAT: now also CHG1.2 (A); no longer CHG1.A
- net D+: now also CN70.2 (D+); no longer CN70.D+
- net D-: now also CN70.3 (D-); no longer CN70.D-
- net D11: now also J10.18 (Pin_18), J11.18 (Pin_18)
- net D12: no longer U4.1 (#IRQ)
- net D2: now also J10.17 (Pin_17), J11.17 (Pin_17), R60.1; no longer D600.2 (DIN)
- net D3: now also U4.1 (#IRQ), J10.14 (Pin_14), J11.14 (Pin_14)
- net D4: no longer U71.4 (EN1)
- net D5: now also R24.2
- net D6: now also R23.2
- net D7: now also J10.6 (Pin_6), J11.6 (Pin_6)
- net DMIC1_CLK: now also U9.3 (CLK)
- net DMIC1_L: now also U9.4 (DOUT)
- net GND: now also CN70.5 (GND), CN70.6 (GND), D10.1 (C), U1.49 (GND), C30.2, C51.1, C90.2, C91.2, J10.19 (Pin_19), J10.20 (Pin_20), J11.19 (Pin_19), J11.20 (Pin_20), J80.3 (Pin_3), R25.1, R26.1, U9.5 (GND), U9.6 (GND), U9.7 (GND), U9.8 (GND); no longer CN70.BASE@1 (GND), D10.C
- net GNDA: now also C810.2, C89.2, J10.5 (Pin_5), J11.5 (Pin_5), J80.4 (Pin_4), J81.4 (Pin_4), U8.11 (PGND), U8.13 (EP), U8.6 (SGND)
- net GPIO0: now also R25.2
- net GPIO1: now also R26.2
- net L_OUT: now also J80.5 (Pin_5), U8.8 (OUTL)
- net R_OUT: now also J81.5 (Pin_5), U8.7 (OUTR)
- net SCL: now also J10.13 (Pin_13), J11.13 (Pin_13)
- net SDA: now also J10.12 (Pin_12), J11.12 (Pin_12)
- net VBUS: now also D71.1 (C), U3.22 (ADAP_IN), C30.1, C51.2, D72.1 (C), J10.10 (Pin_10), J10.9 (Pin_9), J11.10 (Pin_10), J11.9 (Pin_9); no longer CN70.VBUS, D71.C
- net VDDA: no longer R20.1
- net vs1053_LEFT: now also R80.1, R82.2, J10.1 (Pin_1), J11.1 (Pin_1); no longer R81.1, R83.2
- net vs1053_RIGHT: now also R81.1, R83.2, J10.2 (Pin_2), J11.2 (Pin_2); no longer R80.1, R82.2
- net at R10.2: now also D10.2 (A); no longer D10.A
- net LED_FB: now reaches D50.1 (K), R50.1, U5.5 (FB)
- net LED_FB: now also J5.2 (Pin_2)
- net LED_SW: now reaches C50.1, D50.2 (A), L50.2
- net LED_SW: now also J5.3 (Pin_3)
- net at U72.1 (STAT): now also CHG1.1 (C); no longer CHG1.C
- net at R82.1: now also C82.1
- net at R83.1: now also C83.2
- net at R87.1: now also C87.1
- net at R86.1: now also C86.1
- new net: D600.2 (DIN), R60.2
- new net: C83.1, C87.2, U8.4 (INR)
- new net: C89.1, U8.2 (PVSS), U8.5 (VSS)
- new net: C88.1, U8.1 (C1N)
- new net: C88.2, U8.10 (C1P)
- new net: C82.2, C86.2, U8.3 (INL)
- new net: CN70.1 (VBUS), D72.2 (A)
Other:
- note added: "MIC (9)"
- note added: "Mezzanine connector"
- note added: "POWER LED (5)"
- note added: "TOUCH SLIDER (4)"
- note removed: "Power LED (5)"
- note removed: "Touch Slider (4)"
- moved on the sheet: C11, C80, C81, C84, C85, R10, R80, R81, R82, R83, R84, R85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
