File: V2/electronics/Adafruit-Feather-M0-Basic-Proto-PCB-master/Adafruit Feather M0 Basic rev C.kicad_pcb (KiCad board)
At the start: 2 copper layers, 50.8 x 22.9 mm, 39 parts, among them SW1 SPST_TACT-KMR2, U2 SPX3819-3.3, U3 MCP73831T-2ACI/OT, X1 JSTPH, X2 32.768, X3 microUSB

Commit message: pcb design done 24 04 22
Routing:
- net N$9: vias 1 -> 0
- net N$8: vias 1 -> 0
- net N$6: vias 1 -> 0
- net N$48: vias 1 -> 0
- net N$47: vias 1 -> 0
- net N$46: vias 1 -> 0
- net N$45: vias 1 -> 0
- net N$44: vias 1 -> 0
- net N$43: vias 1 -> 0
- net N$42: vias 1 -> 0
- net N$41: vias 1 -> 0
- net N$40: vias 1 -> 0
- net N$39: vias 1 -> 0
- net N$38: vias 1 -> 0
- net N$37: vias 1 -> 0
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