File: V2/electronics/feather vs1053b tests/Adafruit-Music-Maker-FeatherWing-PCB-master/Adafruit VS1053 Headphone FeatherWing.kicad_sch (KiCad schematic)
At the start: 40 parts, among them CN1 2908-05WB-M6, SW1 KMR2, U1 VS1053B, U2 AP7312-1833W6-7, X1 AUDIO_3.5MMJACK_4POL, Y1 ABM8G-12.288MHZ-4Y-T3

Commit message: pcb design done 24 04 22
Connections:
- net 3.3V: now also R16.7 (2); no longer R16.8 (2)
- net GND: now also R16.5 (2), R16.6 (2); no longer R16.8 (2), R16.8 (2)
- net GPIO0: now also R16.4 (1); no longer R16.1
- net GPIO1: now also R16.3 (1); no longer R16.1
- net MP3CS: now also R16.2 (1); no longer R16.1
